Commit message: modify urdf rover

File: src/description/robot_core.xacro (robot description, xacro)
@@ -19,32 +19,32 @@
     <parent link="base_link"/>
     <child link="chassis"/>
-    <origin xyz="-0.1 0 0"/>
+    <origin xyz="-0.15 0 0"/>
 </joint>
 <link name="chassis">
     <visual>
-        <origin xyz="0.15 0 0.075" rpy="0 0 0"/>
+        <origin xyz="0.15 0 0.045" rpy="0 0 0"/>
         <geometry>
-            <box size="0.3 0.3 0.15"/>
+            <box size="0.3 0.2 0.09"/>
         </geometry>
         <material name="white"/>
     </visual>
     <collision>
-        <origin xyz="0.15 0 0.075" rpy="0 0 0"/>
+        <origin xyz="0.15 0 0.045" rpy="0 0 0"/>
         <geometry>
-            <box size="0.3 0.3 0.15"/>
+            <box size="0.3 0.2 0.09"/>
         </geometry>
     </collision>
-    <xacro:inertial_box mass="0.5" x="0.3" y="0.3" z="0.15">
-        <origin xyz="0.15 0 0.075" rpy="0 0 0"/>
+    <xacro:inertial_box mass="0.5" x="0.3" y="0.2" z="0.09">
+        <origin xyz="0.15 0 0.045" rpy="0 0 0"/>
     </xacro:inertial_box>
 </link>
-<!-- LEFT WHEEL -->
-<joint name="left_wheel_joint" type="continuous">
+<!-- REAR LEFT WHEEL -->
+<joint name="front_left_wheel_joint" type="continuous">
     <parent link="base_link"/>
-    <child link="left_wheel"/>
-    <origin xyz="0 0.175 0" rpy="-${pi/2} 0 0"/>
+    <child link="front_left_wheel"/>
+    <origin xyz="-0.13 0.125 0.02" rpy="-${pi/2} 0 0"/>
     <axis xyz="0 0 1"/>
 </joint>
-<link name="left_wheel">
+<link name="front_left_wheel">
     <visual>
         <geometry>
@@ -57,12 +57,12 @@
     </xacro:inertial_cylinder>
 </link>
-<!-- RIGHT WHEEL -->
-<joint name="right_wheel_joint" type="continuous">
+<!-- REAR RIGHT WHEEL -->
+<joint name="front_right_wheel_joint" type="continuous">
     <parent link="base_link"/>
-    <child link="right_wheel"/>
-    <origin xyz="0 -0.175 0" rpy="${pi/2} 0 0"/>
+    <child link="front_right_wheel"/>
+    <origin xyz="-0.13 -0.125 0.02" rpy="${pi/2} 0 0"/>
     <axis xyz="0 0 -1"/>
 </joint>
-<link name="right_wheel">
+<link name="front_right_wheel">
     <visual>
         <geometry>
@@ -75,20 +75,62 @@
     </xacro:inertial_cylinder>
 </link>
-<!-- CASTER WHEEL -->
-<joint name="caster_wheel_joint" type="fixed">
-    <parent link="chassis"/>
-    <child link="caster_wheel"/>
-    <origin xyz="0.24 0 0" rpy="0 0 0"/>
+<!-- FRONT LEFT WHEEL -->
+<joint name="rear_left_wheel_joint" type="continuous">
+    <parent link="base_link"/>
+    <child link="rear_left_wheel"/>
+    <origin xyz="0.13 0.125 0.02" rpy="-${pi/2} 0 0"/>
+    <axis xyz="0 0 1"/>
 </joint>
-<link name="caster_wheel">
+<link name="rear_left_wheel">
     <visual>
         <geometry>
-            <sphere radius="0.05" />
+            <cylinder length="0.04" radius="0.05" />
         </geometry>
-        <material name="black"/>
+        <material name="blue"/>
     </visual>
-    <xacro:inertial_sphere mass="0.1" radius="0.05">
+    <xacro:inertial_cylinder mass="0.1" length="0.05" radius="0.05">
         <origin xyz="0 0 0" rpy="0 0 0"/>
-    </xacro:inertial_sphere>
+    </xacro:inertial_cylinder>
+</link>
+<!-- FRONT RIGHT WHEEL -->
+<joint name="rear_right_wheel_joint" type="continuous">
+    <parent link="base_link"/>
+    <child link="rear_right_wheel"/>
+    <origin xyz="0.13 -0.125 0.02" rpy="${pi/2} 0 0"/>
+    <axis xyz="0 0 -1"/>
+</joint>
+<link name="rear_right_wheel">
+    <visual>
+        <geometry>
+            <cylinder length="0.04" radius="0.05" />
+        </geometry>
+        <material name="blue"/>
+    </visual>
+    <xacro:inertial_cylinder mass="0.1" length="0.05" radius="0.05">
+        <origin xyz="0 0 0" rpy="0 0 0"/>
+    </xacro:inertial_cylinder>
+</link>
+<joint name="arm_base_link" type="fixed">
+    <parent link="base_link"/>
+    <child link="arm_base"/>
+    <origin xyz="0.05 0 0.045"/>
+</joint>
+<link name="arm_base">
+    <visual>
+        <origin xyz="0.05 0 0.045" rpy="0 0 0"/>
+        <geometry>
+            <box size="0.12 0.12 0.005"/>
+        </geometry>
+        <material name="blue"/>
+    </visual>
+    <collision>
+        <origin xyz="0.05 0 0.045" rpy="0 0 0"/>
+        <geometry>
+            <box size="0.12 0.12 0.005"/>
+        </geometry>
+    </collision>
+    <xacro:inertial_box mass="0.5" x="0.12" y="0.12" z="0.005">
+        <origin xyz="0.05 0 0.045" rpy="0 0 0"/>
+    </xacro:inertial_box>
 </link>
 </robot>

Commit message: Added robotic arm URDF

File: src/description/robot_core.xacro (robot description, xacro)
@@ -49,4 +49,5 @@
     <visual>
         <geometry>
+            <!-- <mesh filename="package://articubot_one/meshes/Right_wheel.stl" scale="1 1 1"/> -->
             <cylinder length="0.04" radius="0.05" />
         </geometry>
@@ -111,26 +112,140 @@
     </xacro:inertial_cylinder>
 </link>
+<!-- ROBOTIC ARM -->
+<!-- ARM BASE -->
 <joint name="arm_base_link" type="fixed">
     <parent link="base_link"/>
     <child link="arm_base"/>
-    <origin xyz="0.05 0 0.045"/>
+    <origin xyz="0.05 0 0.09"/>
 </joint>
 <link name="arm_base">
     <visual>
-        <origin xyz="0.05 0 0.045" rpy="0 0 0"/>
-        <geometry>
-            <box size="0.12 0.12 0.005"/>
-        </geometry>
-        <material name="blue"/>
-    </visual>
-    <collision>
-        <origin xyz="0.05 0 0.045" rpy="0 0 0"/>
-        <geometry>
-            <box size="0.12 0.12 0.005"/>
+        <origin xyz="0 0 0" rpy="0 0 0"/>
+        <geometry>
+            <box size="0.12 0.12 0.001"/>
+        </geometry>
+        <material name="blue"/>
+    </visual>
+    <collision>
+        <origin xyz="0 0 0" rpy="0 0 0"/>
+        <geometry>
+            <box size="0.12 0.12 0.001"/>
         </geometry>
     </collision>
     <xacro:inertial_box mass="0.5" x="0.12" y="0.12" z="0.005">
-        <origin xyz="0.05 0 0.045" rpy="0 0 0"/>
+        <origin xyz="0 0 0" rpy="0 0 0"/>
     </xacro:inertial_box>
 </link>
+<!-- ARM JOINT1 -->
+<joint name="arm_joint_1" type="continuous">
+    <parent link="arm_base"/>
+    <child link="arm_link_1"/>
+    <origin xyz="0 0 0.095" rpy="0 0 0"/>
+    <axis xyz="0 0 1"/>
+</joint>
+<link name="arm_link_1">
+    <visual>
+    <origin xyz="0 0 -0.0475" rpy="0 0 0"/>
+        <geometry>
+            <cylinder length="0.095" radius="0.05" />
+        </geometry>
+        <material name="orange"/>
+    </visual>
+    <collision>
+    <origin xyz="0 0 -0.0275" rpy="0 0 0"/>
+        <geometry>
+            <cylinder length="0.055" radius="0.05" />
+        </geometry>
+    </collision>
+    <xacro:inertial_cylinder mass="0.1" length="0.055" radius="0.05">
+    <origin xyz="0 0 -0.0275" rpy="0 0 0"/>
+    </xacro:inertial_cylinder>
+</link>
+<!-- ARM JOINT2 -->
+<joint name="arm_joint_2" type="revolute">
+    <parent link="arm_link_1"/>
+    <child link="arm_link_2"/>
+    <origin xyz="0 0 0" rpy="${pi/2} 0 0"/>
+    <limit effort="30" velocity="1.0" lower="${pi/3}" upper="-${pi/3}"/>
+    <axis xyz="0 0 -1"/>
+</joint>
+<link name="arm_link_2">
+    <visual>
+    <origin xyz="0 0.07 0" rpy="-${pi/2} 0 0"/>
+        <geometry>
+            <cylinder length="0.14" radius="0.04" />
+        </geometry>
+        <material name="blue"/>
+    </visual>
+    <collision>
+    <origin xyz="0 0.07 0" rpy="-${pi/2} 0 0"/>
+        <geometry>
+            <cylinder length="0.14" radius="0.04" />
+        </geometry>
+    </collision>
+    <xacro:inertial_cylinder mass="0.1" length="0.14" radius="0.04">
+    <origin xyz="0 0.07 0" rpy="-${pi/2} 0 0"/>
+    </xacro:inertial_cylinder>
+</link>
+<!-- ARM JOINT3 -->
+<joint name="arm_joint_3" type="revolute">
+    <parent link="arm_link_2"/>
+    <child link="arm_link_3"/>
+    <origin xyz="0 0.14 0" rpy="0 0 0"/>
+    <limit effort="30" velocity="1.0" lower="${pi/3}" upper="-${pi/3}"/>
+    <axis xyz="0 0 -1"/>
+</joint>
+<link name="arm_link_3">
+    <visual>
+    <origin xyz="0 0.06 0" rpy="-${pi/2} 0 0"/>
+        <geometry>
+            <cylinder length="0.12" radius="0.035" />
+        </geometry>
+        <material name="orange"/>
+    </visual>
+    <collision>
+    <origin xyz="0 0.06 0" rpy="-${pi/2} 0 0"/>
+        <geometry>
+            <cylinder length="0.12" radius="0.035" />
+        </geometry>
+    </collision>
+    <xacro:inertial_cylinder mass="0.1" length="0.12" radius="0.035">
+    <origin xyz="0 0.05 0" rpy="-${pi/2} 0 0"/>
+    </xacro:inertial_cylinder>
+</link>
+<!-- ARM JOINT4 -->
+<joint name="arm_joint_4" type="revolute">
+    <parent link="arm_link_3"/>
+    <child link="arm_link_4"/>
+    <origin xyz="0 0.12 0" rpy="-${pi/2} 0 0"/>
+    <limit effort="30" velocity="1.0" lower="${pi/3}" upper="-${pi/3}"/>
+    <axis xyz="0 0 -1"/>
+</joint>
+<link name="arm_link_4">
+    <visual>
+    <origin xyz="0 0 0.04" rpy="0 0 0"/>
+        <geometry>
+            <cylinder length="0.08" radius="0.03" />
+        </geometry>
+        <material name="blue"/>
+    </visual>
+    <collision>
+    <origin xyz="0 0 0.04" rpy="0 0 0"/>
+        <geometry>
+            <cylinder length="0.08" radius="0.03" />
+        </geometry>
+    </collision>
+    <xacro:inertial_cylinder mass="0.1" length="0.08" radius="0.03">
+    <origin xyz="0 0 0.04" rpy="0 0 0"/>
+    </xacro:inertial_cylinder>
+</link>
+<!-- TCP -->
+<joint name="TCP_joint" type="fixed">
+    <parent link="arm_link_4"/>
+    <child link="TCP_link"/>
+    <origin xyz="0 0 0.08" rpy="0 0 0"/>
+    <axis xyz="0 0 1"/>
+</joint>
+<link name="TCP_link">
+</link>
 </robot>

Commit message: urdf completed

File: src/description/robot_core.xacro (robot description, xacro)
@@ -49,5 +49,5 @@
     <visual>
         <geometry>
-            <!-- <mesh filename="package://articubot_one/meshes/Right_wheel.stl" scale="1 1 1"/> -->
+            <!-- <mesh meshfile="package://articubot_one/meshes/Right_wheel.stl" scale="1 1 1"/> -->
             <cylinder length="0.04" radius="0.05" />
         </geometry>
@@ -148,4 +148,5 @@
     <origin xyz="0 0 -0.0475" rpy="0 0 0"/>
         <geometry>
+            <!-- <mesh filename="/home/ubuntu/Desktop/Project/articubot_one/src/meshes/arm_base.STL" scale="1 1 1"/> -->
             <cylinder length="0.095" radius="0.05" />
         </geometry>
@@ -168,5 +169,5 @@
     <origin xyz="0 0 0" rpy="${pi/2} 0 0"/>
     <limit effort="30" velocity="1.0" lower="${pi/3}" upper="-${pi/3}"/>
-    <axis xyz="0 0 -1"/>
+    <axis xyz="0 0 1"/>
 </joint>
 <link name="arm_link_2">
@@ -194,5 +195,5 @@
     <origin xyz="0 0.14 0" rpy="0 0 0"/>
     <limit effort="30" velocity="1.0" lower="${pi/3}" upper="-${pi/3}"/>
-    <axis xyz="0 0 -1"/>
+    <axis xyz="0 0 1"/>
 </joint>
 <link name="arm_link_3">
@@ -224,17 +225,43 @@
 <link name="arm_link_4">
     <visual>
+    <origin xyz="0 0 0.03" rpy="0 0 0"/>
+        <geometry>
+            <cylinder length="0.06" radius="0.03" />
+        </geometry>
+        <material name="blue"/>
+    </visual>
+    <collision>
+    <origin xyz="0 0 0.03" rpy="0 0 0"/>
+        <geometry>
+            <cylinder length="0.06" radius="0.03" />
+        </geometry>
+    </collision>
+    <xacro:inertial_cylinder mass="0.1" length="0.06" radius="0.03">
+    <origin xyz="0 0 0.03" rpy="0 0 0"/>
+    </xacro:inertial_cylinder>
+</link>
+<!-- ARM JOINT5 -->
+<joint name="arm_joint_5" type="revolute">
+    <parent link="arm_link_4"/>
+    <child link="arm_link_5"/>
+    <origin xyz="0 0 0.06" rpy="${pi/2} 0 0"/>
+    <limit effort="30" velocity="1.0" lower="${pi/3}" upper="-${pi/3}"/>
+    <axis xyz="0 0 1"/>
+</joint>
+<link name="arm_link_5">
+    <visual>
+    <origin xyz="0 0.04 0" rpy="${pi/2} 0 0"/>
+        <geometry>
+            <cylinder length="0.08" radius="0.025" />
+        </geometry>
+        <material name="orange"/>
+    </visual>
+    <collision>
     <origin xyz="0 0 0.04" rpy="0 0 0"/>
         <geometry>
-            <cylinder length="0.08" radius="0.03" />
-        </geometry>
-        <material name="blue"/>
-    </visual>
-    <collision>
-    <origin xyz="0 0 0.04" rpy="0 0 0"/>
-        <geometry>
-            <cylinder length="0.08" radius="0.03" />
-        </geometry>
-    </collision>
-    <xacro:inertial_cylinder mass="0.1" length="0.08" radius="0.03">
+            <cylinder length="0.08" radius="0.025" />
+        </geometry>
+    </collision>
+    <xacro:inertial_cylinder mass="0.1" length="0.08" radius="0.025">
     <origin xyz="0 0 0.04" rpy="0 0 0"/>
     </xacro:inertial_cylinder>
@@ -242,7 +269,7 @@
 <!-- TCP -->
 <joint name="TCP_joint" type="fixed">
-    <parent link="arm_link_4"/>
+    <parent link="arm_link_5"/>
     <child link="TCP_link"/>
-    <origin xyz="0 0 0.08" rpy="0 0 0"/>
+    <origin xyz="0 0.08 0" rpy="0 0 0"/>
     <axis xyz="0 0 1"/>
 </joint>

Commit message: adjust urdf model

File: src/description/robot_core.xacro (robot description, xacro)
@@ -258,5 +258,5 @@
     </visual>
     <collision>
-    <origin xyz="0 0 0.04" rpy="0 0 0"/>
+    <origin xyz="0 0.04 0" rpy="${pi/2} 0 0"/>
         <geometry>
             <cylinder length="0.08" radius="0.025" />
@@ -264,5 +264,5 @@
     </collision>
     <xacro:inertial_cylinder mass="0.1" length="0.08" radius="0.025">
-    <origin xyz="0 0 0.04" rpy="0 0 0"/>
+        <origin xyz="0 0.04 0" rpy="${pi/2} 0 0"/>
     </xacro:inertial_cylinder>
 </link>

Commit message: fixed color in gazebo

File: src/description/robot_core.xacro (robot description, xacro)
@@ -39,4 +39,7 @@
     </xacro:inertial_box>
 </link>
+<gazebo reference="chassis">
+    <material>Gazebo/White</material>
+</gazebo>
 <!-- REAR LEFT WHEEL -->
 <joint name="front_left_wheel_joint" type="continuous">
@@ -58,4 +61,7 @@
     </xacro:inertial_cylinder>
 </link>
+<gazebo reference="front_left_wheel">
+    <material>Gazebo/Blue</material>
+</gazebo>
 <!-- REAR RIGHT WHEEL -->
 <joint name="front_right_wheel_joint" type="continuous">
@@ -76,4 +82,7 @@
     </xacro:inertial_cylinder>
 </link>
+<gazebo reference="front_right_wheel">
+    <material>Gazebo/Blue</material>
+</gazebo>
 <!-- FRONT LEFT WHEEL -->
 <joint name="rear_left_wheel_joint" type="continuous">
@@ -94,4 +103,7 @@
     </xacro:inertial_cylinder>
 </link>
+<gazebo reference="rear_left_wheel">
+    <material>Gazebo/Blue</material>
+</gazebo>
 <!-- FRONT RIGHT WHEEL -->
 <joint name="rear_right_wheel_joint" type="continuous">
@@ -112,4 +124,7 @@
     </xacro:inertial_cylinder>
 </link>
+<gazebo reference="rear_right_wheel">
+    <material>Gazebo/Blue</material>
+</gazebo>
 <!-- ROBOTIC ARM -->
 <!-- ARM BASE -->
@@ -137,4 +152,7 @@
     </xacro:inertial_box>
 </link>
+<gazebo reference="arm_base">
+    <material>Gazebo/Blue</material>
+</gazebo>
 <!-- ARM JOINT1 -->
 <joint name="arm_joint_1" type="continuous">
@@ -163,4 +181,7 @@
     </xacro:inertial_cylinder>
 </link>
+<gazebo reference="arm_link_1">
+    <material>Gazebo/Orange</material>
+</gazebo>
 <!-- ARM JOINT2 -->
 <joint name="arm_joint_2" type="revolute">
@@ -189,4 +210,7 @@
     </xacro:inertial_cylinder>
 </link>
+<gazebo reference="arm_link_2">
+    <material>Gazebo/Blue</material>
+</gazebo>
 <!-- ARM JOINT3 -->
 <joint name="arm_joint_3" type="revolute">
@@ -215,4 +239,7 @@
     </xacro:inertial_cylinder>
 </link>
+<gazebo reference="arm_link_3">
+    <material>Gazebo/Orange</material>
+</gazebo>
 <!-- ARM JOINT4 -->
 <joint name="arm_joint_4" type="revolute">
@@ -241,4 +268,7 @@
     </xacro:inertial_cylinder>
 </link>
+<gazebo reference="arm_link_4">
+    <material>Gazebo/Blue</material>
+</gazebo>
 <!-- ARM JOINT5 -->
 <joint name="arm_joint_5" type="revolute">
@@ -267,4 +297,7 @@
     </xacro:inertial_cylinder>
 </link>
+<gazebo reference="arm_link_5">
+    <material>Gazebo/Orange</material>
+</gazebo>
 <!-- TCP -->
 <joint name="TCP_joint" type="fixed">
